File: Schmatic_eagle/schematic2.sch (EAGLE design)
At the start: 6 parts, among them IC1 MEGA16-A, IC2 MC145027DW

Commit message: Schematic update
Parts:
- added ANT1: (no value), discrete:ANTENNA
- added M1: WIRELESS-XY-MK-5V, diy-modules:WIRELESS-XY-MK-5V
Connections:
- new net N$13: IC2G$1.DIN, M1.DATA.1
- new net N$15: ANT1.1, M1.ANT
- new net VCC: M1.VCC
- net GND: now also M1.GND
Changed lines of the file:
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@@
 <layer number="97" name="Info" color="7" fill="1" visible="yes" active="yes"/>
 <layer number="98" name="Guide" color="6" fill="1" visible="yes" active="yes"/>
+<layer number="101" name="Hidden" color="15" fill="1" visible="yes" active="yes"/>
+<layer number="102" name="Changes" color="12" fill="1" visible="yes" active="yes"/>
 </layers>
 <schematic xreflabel="%F%N/%S.%C%R" xrefpart="/%S.%C%R">
@@
 <part name="C2" library="rcl" library_urn="urn:adsk.eagle:library:334" deviceset="C-EU" device="C0805" package3d_urn="urn:adsk.eagle:package:23617/2" value="910pF"/>
 <part name="R2" library="rcl" library_urn="urn:adsk.eagle:library:334" deviceset="R-EU_" device="01005" package3d_urn="urn:adsk.eagle:package:26133/2" value="100k"/>
+<part name="M1" library="diy-modules" deviceset="WIRELESS-XY-MK-5V" device=""/>
+<part name="SUPPLY2" library="supply2" library_urn="urn:adsk.eagle:library:372" deviceset="GND" device=""/>
+<part name="P+1" library="supply1" library_urn="urn:adsk.eagle:library:371" deviceset="VCC" device=""/>
+<part name="ANT1" library="discrete" library_urn="urn:adsk.eagle:library:211" deviceset="ANTENNA" device="" package3d_urn="urn:adsk.eagle:package:12928/1"/>
 </parts>
 <sheets>
@@
 <attribute name="NAME" x="161.29" y="52.2986" size="1.778" layer="95"/>
 <attribute name="VALUE" x="163.83" y="51.562" size="1.778" layer="96" rot="R180"/>
+</instance>
+<instance part="M1" gate="G$1" x="139.7" y="-7.62" smashed="yes" rot="R90">
+<attribute name="NAME" x="121.92" y="-17.78" size="1.778" layer="95" rot="R90"/>
+<attribute name="VALUE" x="124.46" y="-17.78" size="1.778" layer="96" rot="R90"/>
+</instance>
+<instance part="SUPPLY2" gate="GND" x="106.68" y="-5.08" smashed="yes">
+<attribute name="VALUE" x="104.775" y="-8.255" size="1.778" layer="96"/>
+</instance>
+<instance part="P+1" gate="VCC" x="170.18" y="30.48" smashed="yes">
+<attribute name="VALUE" x="167.64" y="27.94" size="1.778" layer="96" rot="R90"/>
+</instance>
+<instance part="ANT1" gate="A" x="182.88" y="30.48" smashed="yes">
+<attribute name="NAME" x="180.34" y="31.75" size="1.778" layer="95"/>
+<attribute name="VALUE" x="185.42" y="25.4" size="1.778" layer="96"/>
 </instance>
 </instances>
@@
 <junction x="147.32" y="43.18"/>
 </segment>
+<segment>
+<pinref part="M1" gate="G$1" pin="GND"/>
+<pinref part="SUPPLY2" gate="GND" pin="GND"/>
+<wire x1="129.54" y1="7.62" x2="106.68" y2="7.62" width="0.1524" layer="91"/>
+<wire x1="106.68" y1="7.62" x2="106.68" y2="-2.54" width="0.1524" layer="91"/>
+</segment>
 </net>
 <net name="N$12" class="0">
@@
 </segment>
 </net>
+<net name="N$13" class="0">
+<segment>
+<pinref part="IC2" gate="G$1" pin="DIN"/>
+<pinref part="M1" gate="G$1" pin="DATA.1"/>
+<wire x1="132.08" y1="58.42" x2="132.08" y2="7.62" width="0.1524" layer="91"/>
+</segment>
+</net>
+<net name="VCC" class="0">
+<segment>
+<pinref part="M1" gate="G$1" pin="VCC"/>
+<wire x1="137.16" y1="7.62" x2="137.16" y2="20.32" width="0.1524" layer="91"/>
+<wire x1="137.16" y1="20.32" x2="170.18" y2="20.32" width="0.1524" layer="91"/>
+<pinref part="P+1" gate="VCC" pin="VCC"/>
+<wire x1="170.18" y1="20.32" x2="170.18" y2="27.94" width="0.1524" layer="91"/>
+</segment>
+</net>
+<net name="N$15" class="0">
+<segment>
+<pinref part="M1" gate="G$1" pin="ANT"/>
+<pinref part="ANT1" gate="A" pin="1"/>
+<wire x1="149.86" y1="7.62" x2="182.88" y2="7.62" width="0.1524" layer="91"/>
+<wire x1="182.88" y1="7.62" x2="182.88" y2="25.4" width="0.1524" layer="91"/>
+</segment>
+</net>

Commit message: Schematic 2 updates
Parts:
- added R3: 1k, rcl:R-EU_M0805
- added S1: RDT1034, switch:RDT1034
- added SV1: (no value), con-amp-mt:L05P
Connections:
- new net N$14: IC1.(SCK)PB7, SV1-5.S
- new net N$16: IC1.(MISO)PB6, SV1-4.S
- new net N$17: IC1.(MOSI)PB5, SV1-3.S
- new net N$18: IC1.(SS)PB4, SV1-2.S
- new net N$19: IC1.RESET, R3.2, S1.A1
- net GND: now also IC1.GND, IC1.GND1, IC1.GND2, IC1.GND@1, S1.B
- net VCC: now also IC1.AREF, IC1.AVCC, IC1.VCC, IC1.VCC1, IC1.VCC2, R3.1
Other:
- moved on the sheet: IC1

Commit message: Schematic 2 updates
Parts:
- added DIS1: EA_DIP, display-lcd:EA_DIP
- added U$1: LCD-I2C-CONVERTER, diy-modules:LCD-I2C-CONVERTER
Connections:
- new net N$20: IC1.(ADC4)PA4, IC2G$1.VT
- new net N$21: IC1.PC0(SCL), U$1.SCL
- new net N$22: IC1.PC1(SDA), U$1.SDA
- new net N$23: DIS1.D0, U$1.DB0
- new net N$24: DIS1.RS, U$1.RS
- new net N$26: DIS1.R/W, U$1.R/W
- new net N$27: DIS1.E, U$1.EN
- new net N$28: DIS1.D1, U$1.DB1
- new net N$29: DIS1.D2, U$1.DB2
- new net N$30: DIS1.D3, U$1.DB3
- new net N$31: DIS1.D4, U$1.DB4
- new net N$32: DIS1.D5, U$1.DB5
- new net N$33: DIS1.VDD, U$1.VDD
- new net N$34: DIS1.D6, U$1.DB6
- new net N$36: DIS1.A, U$1.LED.A
- new net N$37: DIS1.C, U$1.LED.K
- new net N$38: DIS1.D7, U$1.DB7
- net GND: now also DIS1.VSS, U$1.GND, U$1.VSS
- net N$13: now also M1.DATA.2
- net VCC: now also DIS1.VEE, U$1.VCC, U$1.VEE
Other:
- moved on the sheet: SV1-1

Commit message: Schematic 2 updates
Parts:
- added C3: 0.1uF, rcl:C-EUC0805
- added J1: (no value), con-amp:MTA02-156
Connections:
- net GND: now also C3.2, J1.2
- net VCC: now also C3.1, J1.1
Changed lines of the file:
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@@
 <part name="U$1" library="diy-modules" deviceset="LCD-I2C-CONVERTER" device=""/>
 <part name="P+3" library="supply1" library_urn="urn:adsk.eagle:library:371" deviceset="VCC" device=""/>
+<part name="J1" library="con-amp" library_urn="urn:adsk.eagle:library:127" deviceset="MTA02-156" device="" package3d_urn="urn:adsk.eagle:package:8081562/1"/>
+<part name="SUPPLY5" library="supply2" library_urn="urn:adsk.eagle:library:372" deviceset="GND" device=""/>
+<part name="P+4" library="supply1" library_urn="urn:adsk.eagle:library:371" deviceset="VCC" device=""/>
+<part name="C3" library="rcl" library_urn="urn:adsk.eagle:library:334" deviceset="C-EU" device="C0805" package3d_urn="urn:adsk.eagle:package:23617/2" value="0.1uF"/>
 </parts>
 <sheets>
@@
 <instance part="P+3" gate="VCC" x="88.9" y="-50.8" smashed="yes">
 <attribute name="VALUE" x="86.36" y="-53.34" size="1.778" layer="96" rot="R90"/>
+</instance>
+<instance part="J1" gate="G$1" x="147.32" y="114.3" smashed="yes">
+<attribute name="NAME" x="152.4" y="114.3" size="1.778" layer="95"/>
+<attribute name="VALUE" x="152.4" y="110.49" size="1.778" layer="96"/>
+</instance>
+<instance part="SUPPLY5" gate="GND" x="162.56" y="104.14" smashed="yes">
+<attribute name="VALUE" x="160.655" y="100.965" size="1.778" layer="96"/>
+</instance>
+<instance part="P+4" gate="VCC" x="137.16" y="116.84" smashed="yes">
+<attribute name="VALUE" x="134.62" y="114.3" size="1.778" layer="96" rot="R90"/>
+</instance>
+<instance part="C3" gate="G$1" x="147.32" y="93.98" smashed="yes" rot="R90">
+<attribute name="NAME" x="146.939" y="95.504" size="1.778" layer="95" rot="R90"/>
+<attribute name="VALUE" x="152.019" y="95.504" size="1.778" layer="96" rot="R90"/>
 </instance>
 </instances>
@@
 <pinref part="SUPPLY4" gate="GND" pin="GND"/>
 <wire x1="45.72" y1="121.92" x2="45.72" y2="119.38" width="0.1524" layer="91"/>
+</segment>
+<segment>
+<pinref part="J1" gate="G$1" pin="2"/>
+<wire x1="149.86" y1="111.76" x2="149.86" y2="106.68" width="0.1524" layer="91"/>
+<pinref part="SUPPLY5" gate="GND" pin="GND"/>
+<wire x1="149.86" y1="106.68" x2="154.94" y2="106.68" width="0.1524" layer="91"/>
+<pinref part="C3" gate="G$1" pin="2"/>
+<wire x1="154.94" y1="106.68" x2="162.56" y2="106.68" width="0.1524" layer="91"/>
+<wire x1="152.4" y1="93.98" x2="154.94" y2="93.98" width="0.1524" layer="91"/>
+<wire x1="154.94" y1="93.98" x2="154.94" y2="106.68" width="0.1524" layer="91"/>
+<junction x="154.94" y="106.68"/>
 </segment>
 </net>
@@
 <junction x="78.74" y="-60.96"/>
 </segment>
-</net>
+<segment>
+<pinref part="P+4" gate="VCC" pin="VCC"/>
+<wire x1="137.16" y1="114.3" x2="137.16" y2="106.68" width="0.1524" layer="91"/>
+<wire x1="137.16" y1="106.68" x2="139.7" y2="106.68" width="0.1524" layer="91"/>
+<pinref part="J1" gate="G$1" pin="1"/>
+<wire x1="139.7" y1="106.68" x2="147.32" y2="106.68" width="0.1524" layer="91"/>
+<wire x1="147.32" y1="106.68" x2="147.32" y2="111.76" width="0.1524" layer="91"/>
+<pinref part="C3" gate="G$1" pin="1"/>
+<wire x1="144.78" y1="93.98" x2="139.7" y2="93.98" width="0.1524" layer="91"/>
+<wire x1="139.7" y1="93.98" x2="139.7" y2="106.68" width="0.1524" layer="91"/>
+<junction x="139.7" y="106.68"/>
+</segment>
+</net>

Commit message: Schematic 2 updates
Parts:
- R1, R2: device rcl:R-EU_01005 -> rcl:R-EU_R0805
Changed lines of the file:
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@@
 <layer number="18" name="Vias" color="2" fill="1" visible="yes" active="no"/>
 <layer number="19" name="Unrouted" color="6" fill="1" visible="yes" active="no"/>
-<layer number="20" name="Dimension" color="15" fill="1" visible="yes" active="no"/>
+<layer number="20" name="Dimension" color="24" fill="1" visible="yes" active="no"/>
 <layer number="21" name="tPlace" color="7" fill="1" visible="yes" active="no"/>
 <layer number="22" name="bPlace" color="7" fill="1" visible="yes" active="no"/>
@@
 <part name="IC2" library="micro-motorola" library_urn="urn:adsk.eagle:library:289" deviceset="MC145027" device="DW" package3d_urn="urn:adsk.eagle:package:19965/1"/>
 <part name="IC1" library="atmel" library_urn="urn:adsk.eagle:library:105" deviceset="MEGA16" device="-A" package3d_urn="urn:adsk.eagle:package:4319/1"/>
-<part name="R1" library="rcl" library_urn="urn:adsk.eagle:library:334" deviceset="R-EU_" device="01005" package3d_urn="urn:adsk.eagle:package:26133/2" value="10k"/>
+<part name="R1" library="rcl" library_urn="urn:adsk.eagle:library:334" deviceset="R-EU_" device="R0805" package3d_urn="urn:adsk.eagle:package:23553/2" value="10k"/>
 <part name="C1" library="rcl" library_urn="urn:adsk.eagle:library:334" deviceset="C-EU" device="C0805" package3d_urn="urn:adsk.eagle:package:23617/2" value="470pF"/>
 <part name="SUPPLY1" library="supply2" library_urn="urn:adsk.eagle:library:372" deviceset="GND" device=""/>
 <part name="C2" library="rcl" library_urn="urn:adsk.eagle:library:334" deviceset="C-EU" device="C0805" package3d_urn="urn:adsk.eagle:package:23617/2" value="910pF"/>
-<part name="R2" library="rcl" library_urn="urn:adsk.eagle:library:334" deviceset="R-EU_" device="01005" package3d_urn="urn:adsk.eagle:package:26133/2" value="100k"/>
+<part name="R2" library="rcl" library_urn="urn:adsk.eagle:library:334" deviceset="R-EU_" device="R0805" package3d_urn="urn:adsk.eagle:package:23553/2" value="100k"/>
 <part name="M1" library="diy-modules" deviceset="WIRELESS-XY-MK-5V" device=""/>
 <part name="SUPPLY2" library="supply2" library_urn="urn:adsk.eagle:library:372" deviceset="GND" device=""/>
