File: Schmatic_eagle/schematic2.brd (EAGLE design)
At the start: 100 x 80 mm, 15 parts, among them IC1 MEGA16-A, IC2 MC145027DW, M1 WIRELESS-XY-MK-5V

Commit message: Schematic 2 updates
Routing:
- net N$37: track 85.5 -> 87.3 mm
- net N$27: track 119.7 -> 118.6 mm
- added copper zone on layer 1, net GND
Other:
- board text added: "SS"
- board text removed: "MISO"
- board text removed: "MOSI"
- board text removed: "SCK"
- board text removed: "ss"
Changed lines of the file:
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@@
 <wire x1="100" y1="80" x2="0" y2="80" width="0" layer="20"/>
 <wire x1="0" y1="80" x2="0" y2="0" width="0" layer="20"/>
-<text x="21.59" y="55.88" size="1.778" layer="16" rot="MR0">+VCC</text>
-<text x="22.86" y="71.12" size="1.778" layer="16" rot="MR0">ss</text>
-<text x="26.67" y="68.58" size="1.778" layer="16" rot="MR0">MOSI</text>
-<text x="26.67" y="66.04" size="1.778" layer="16" rot="MR0">MISO</text>
-<text x="26.67" y="63.5" size="1.778" layer="16" rot="MR0">SCK</text>
+<text x="22.86" y="55.88" size="1.778" layer="16" font="vector" rot="MR0">+VCC</text>
+<text x="25.4" y="71.12" size="1.778" layer="16" rot="MR0">SS</text>
 </plain>
 <attributes>
@@
 <via x="52.07" y="50.165" extent="1-16" drill="0.35"/>
 <via x="52.07" y="45.72" extent="1-16" drill="0.35"/>
+<polygon width="0.3048" layer="1" rank="6">
+<vertex x="2.54" y="78.74"/>
+<vertex x="2.54" y="3.81"/>
+<vertex x="5.08" y="1.27"/>
+<vertex x="95.25" y="1.27"/>
+<vertex x="96.52" y="2.54"/>
+<vertex x="97.79" y="3.81"/>
+<vertex x="97.79" y="76.2"/>
+<vertex x="95.25" y="78.74"/>
+<vertex x="93.98" y="78.74"/>
+</polygon>
 </signal>
 <signal name="N$12">
@@
 <wire x1="41.75125" y1="48.10125" x2="46.19625" y2="48.10125" width="0.1524" layer="1"/>
 <wire x1="36.195" y1="48.10125" x2="41.75125" y2="48.10125" width="0.1524" layer="16"/>
-<wire x1="19.52625" y1="64.77" x2="36.195" y2="48.10125" width="0.1524" layer="16"/>
+<wire x1="36.195" y1="48.10125" x2="19.52625" y2="64.77" width="0.1524" layer="16"/>
 <wire x1="19.05" y1="64.77" x2="19.52625" y2="64.77" width="0.1524" layer="16"/>
 <wire x1="46.19625" y1="48.10125" x2="46.27" y2="48.12" width="0.1524" layer="1"/>
@@
 <wire x1="40.9575" y1="48.73625" x2="46.0375" y2="48.73625" width="0.1524" layer="1"/>
 <wire x1="37.62375" y1="48.73625" x2="40.9575" y2="48.73625" width="0.1524" layer="16"/>
-<wire x1="19.05" y1="67.31" x2="37.62375" y2="48.73625" width="0.1524" layer="16"/>
+<wire x1="37.62375" y1="48.73625" x2="19.05" y2="67.31" width="0.1524" layer="16"/>
 <wire x1="46.19625" y1="48.895" x2="46.27" y2="48.92" width="0.1524" layer="1"/>
 <wire x1="19.05" y1="67.31" x2="18.95" y2="67.35" width="0.1524" layer="16"/>
@@
 <contactref element="DIS1" pad="6"/>
 <wire x1="9.8425" y1="36.98875" x2="21.59" y2="25.24125" width="0.1524" layer="1"/>
-<wire x1="9.8425" y1="63.5" x2="9.8425" y2="36.98875" width="0.1524" layer="1"/>
-<wire x1="40.005" y1="63.5" x2="9.8425" y2="63.5" width="0.1524" layer="1"/>
-<wire x1="53.49875" y1="76.99375" x2="40.005" y2="63.5" width="0.1524" layer="1"/>
-<wire x1="77.94625" y1="76.99375" x2="53.49875" y2="76.99375" width="0.1524" layer="1"/>
-<wire x1="80.01" y1="74.93" x2="77.94625" y2="76.99375" width="0.1524" layer="1"/>
+<wire x1="9.8425" y1="59.69" x2="9.8425" y2="36.98875" width="0.1524" layer="1"/>
+<wire x1="33.655" y1="59.69" x2="9.8425" y2="59.69" width="0.1524" layer="1"/>
+<wire x1="52.22875" y1="78.26375" x2="33.655" y2="59.69" width="0.1524" layer="1"/>
+<wire x1="76.67625" y1="78.26375" x2="52.22875" y2="78.26375" width="0.1524" layer="1"/>
+<wire x1="80.01" y1="74.93" x2="76.67625" y2="78.26375" width="0.1524" layer="1"/>
 <wire x1="21.59" y1="25.24125" x2="21.59" y2="25.24" width="0.1524" layer="1"/>
 </signal>
@@
 <contactref element="U$1" pad="J2.16"/>
 <contactref element="DIS1" pad="18"/>
-<wire x1="83.82" y1="16.51" x2="85.09" y2="15.24" width="0.1524" layer="1"/>
-<wire x1="83.82" y1="55.40375" x2="83.82" y2="16.51" width="0.1524" layer="1"/>
-<wire x1="84.29625" y1="55.40375" x2="83.82" y2="55.40375" width="0.1524" layer="1"/>
+<wire x1="82.55" y1="17.78" x2="85.09" y2="15.24" width="0.1524" layer="1"/>
+<wire x1="82.55" y1="55.40375" x2="82.55" y2="17.78" width="0.1524" layer="1"/>
+<wire x1="84.29625" y1="55.40375" x2="82.55" y2="55.40375" width="0.1524" layer="1"/>
 <wire x1="87.3125" y1="58.42" x2="84.29625" y2="55.40375" width="0.1524" layer="1"/>
 <wire x1="87.3125" y1="59.3725" x2="87.3125" y2="58.42" width="0.1524" layer="1"/>
